File: hardware/lab_boards/5b-to-oscope-daq-board/5b-to-oscope-daq-board.sch (KiCad schematic (older format))
At the start: 18 parts, among them J1 OSCOPE 3, J10 OSCOPE 6, J11 OSCOPE 1, J12 DAQ 6, J13 TX_SHUNT, J14 OSCOPE 7, J15 DAQ 7, J16 OSCOPE 8, J17 5B P1, J18 TO DAQ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

Commit message: Added an AWG to TX array connection and calibration board project
Parts:
- gave numbers to parts that had none: 1
Changed lines of the file:
@@
 Connection ~ 5150 4400
 $Comp
-L Connector:Conn_Coaxial J?
+L Connector:Conn_Coaxial J7
 U 1 1 5F6BCFF9
 P 2700 4650
-F 0 "J?" H 2628 4888 50  0000 C CNN
+F 0 "J7" H 2628 4888 50  0000 C CNN
 F 1 "OSCOPE5" V 2850 4550 50  0000 C CNN
 F 2 "Connector_Coaxial:BNC_Amphenol_B6252HB-NPP3G-50_Horizontal" H 2700 4650 50  0001 C CNN
