File: hardware/lab_boards/awg-tx-shunt/awg-tx-shunt.sch (KiCad schematic (older format))
At the start: 8 parts, among them J1 1984659-phoenix-6pos-1984659, J2 TX OUT, J3 TX-SHUNT, SW1 100DP1T1B1M2QEH, SW2 100DP1T1B1M2QEH

Commit message: Added some notes to the shunt board design.
Parts:
- added H1, H2, H3, H4: MountingHole, MountingHole:MountingHole_3.2mm_M3_Pad_Via, symbol Mechanical:MountingHole
- J2: value TX OUT -> TX ARRAY
Connections:
- net labels added: Earth
Other:
- note added: "CURRENT SHUNT RESISTOR\n3mOhms"
- note added: "shunt?"
- note removed: "CURRENT SHUNT RESISTOR"
Changed lines of the file:
@@
 TX-SHUNT ISOLATION/DIRECT SWITCH
 Text Notes 1450 3000 0    50   ~ 0
-CURRENT SHUNT RESISTOR
+CURRENT SHUNT RESISTOR\n3mOhms
 Wire Wire Line
 	1150 2900 1350 2900
@@
 P 9700 2750
 F 0 "J2" H 9470 2746 50  0000 R CNN
-F 1 "TX OUT" H 9470 2655 50  0000 R CNN
+F 1 "TX ARRAY" H 9470 2655 50  0000 R CNN
 F 2 "amphenol-isolated-pcb-mount-bnc:CONN_1-1337543-0" H 9700 2750 50  0001 L BNN
 F 3 "1" H 9700 2750 50  0001 L BNN
@@
 	-1   0    0    -1
 $EndComp
-$Comp
-L power:GNDPWR #PWR0102
-U 1 1 5F695BC3
-P 9250 3300
-F 0 "#PWR0102" H 9250 3100 50  0001 C CNN
-F 1 "GNDPWR" H 9254 3146 50  0000 C CNN
-F 2 "" H 9250 3250 50  0001 C CNN
-F 3 "" H 9250 3250 50  0001 C CNN
-	1    9250 3300
-	1    0    0    -1
-$EndComp
 Wire Wire Line
 	9400 2750 8950 2750
@@
 Wire Wire Line
 	2600 2800 3600 2800
-$Comp
-L power:GNDPWR #PWR0103
-U 1 1 5F69C7A7
-P 8950 4750
-F 0 "#PWR0103" H 8950 4550 50  0001 C CNN
-F 1 "GNDPWR" H 8954 4596 50  0000 C CNN
-F 2 "" H 8950 4700 50  0001 C CNN
-F 3 "" H 8950 4700 50  0001 C CNN
-	1    8950 4750
-	1    0    0    -1
-$EndComp
 Wire Wire Line
 	8950 4300 8950 4750
@@
 $EndComp
 $Comp
-L 100DP1T1B1M2QEH:100DP1T1B1M2QEH SW1
-U 1 1 5F63DBC1
-P 3800 3300
-F 0 "SW1" H 4200 4567 50  0000 C CNN
-F 1 "100DP1T1B1M2QEH" H 4200 4476 50  0000 C CNN
-F 2 "switches:100DP1T1B1M2QEH" H 3800 3300 50  0001 L BNN
-F 3 "EG2400-ND" H 3800 3300 50  0001 L BNN
-	1    3800 3300
-	1    0    0    -1
-$EndComp
-$Comp
 L awg-tx-shunt-rescue:WSL36373L000FEA-WSL36373L000FEA R1
 U 1 1 5F63D2DC
@@
 Wire Wire Line
 	4800 2900 5850 2900
+$Comp
+L Mechanical:MountingHole H1
+U 1 1 5F63F8E4
+P 2450 6050
+F 0 "H1" H 2550 6096 50  0000 L CNN
+F 1 "MountingHole" H 2550 6005 50  0000 L CNN
+F 2 "MountingHole:MountingHole_3.2mm_M3_Pad_Via" H 2450 6050 50  0001 C CNN
+F 3 "~" H 2450 6050 50  0001 C CNN
+	1    2450 6050
+	1    0    0    -1
+$EndComp
+$Comp
+L Mechanical:MountingHole H2
+U 1 1 5F6472C6
+P 3700 6050
+F 0 "H2" H 3800 6096 50  0000 L CNN
+F 1 "MountingHole" H 3800 6005 50  0000 L CNN
+F 2 "MountingHole:MountingHole_3.2mm_M3_Pad_Via" H 3700 6050 50  0001 C CNN
+F 3 "~" H 3700 6050 50  0001 C CNN
+	1    3700 6050
+	1    0    0    -1
+$EndComp
+$Comp
+L Mechanical:MountingHole H3
+U 1 1 5F64875D
+P 4900 6050
+F 0 "H3" H 5000 6096 50  0000 L CNN
+F 1 "MountingHole" H 5000 6005 50  0000 L CNN
+F 2 "MountingHole:MountingHole_3.2mm_M3_Pad_Via" H 4900 6050 50  0001 C CNN
+F 3 "~" H 4900 6050 50  0001 C CNN
+	1    4900 6050
+	1    0    0    -1
+$EndComp
+$Comp
+L Mechanical:MountingHole H4
+U 1 1 5F649C5A
+P 6000 6050
+F 0 "H4" H 6100 6096 50  0000 L CNN
+F 1 "MountingHole" H 6100 6005 50  0000 L CNN
+F 2 "MountingHole:MountingHole_3.2mm_M3_Pad_Via" H 6000 6050 50  0001 C CNN
+F 3 "~" H 6000 6050 50  0001 C CNN
+	1    6000 6050
+	1    0    0    -1
+$EndComp
+Text Notes 8300 3200 0    50   ~ 0
+shunt?
+$Comp
+L 100DP1T1B1M2QEH:100DP1T1B1M2QEH SW1
+U 1 1 5F63DBC1
+P 3800 3300
+F 0 "SW1" H 4200 4567 50  0000 C CNN
+F 1 "100DP1T1B1M2QEH" H 4200 4476 50  0000 C CNN
+F 2 "switches:100DP1T1B1M2QEH" H 3800 3300 50  0001 L BNN
+F 3 "EG2400-ND" H 3800 3300 50  0001 L BNN
+	1    3800 3300
+	1    0    0    -1
+$EndComp
+$Comp
+L power:Earth #PWR?
+U 1 1 5F675DA7
+P 8950 4750
+F 0 "#PWR?" H 8950 4500 50  0001 C CNN
+F 1 "Earth" H 8950 4600 50  0001 C CNN
+F 2 "" H 8950 4750 50  0001 C CNN
+F 3 "~" H 8950 4750 50  0001 C CNN
+	1    8950 4750
+	1    0    0    -1
+$EndComp
+$Comp
+L power:Earth #PWR?
+U 1 1 5F67ACEC
+P 9250 3300
+F 0 "#PWR?" H 9250 3050 50  0001 C CNN
+F 1 "Earth" H 9250 3150 50  0001 C CNN
+F 2 "" H 9250 3300 50  0001 C CNN
+F 3 "~" H 9250 3300 50  0001 C CNN
+	1    9250 3300
+	1    0    0    -1
+$EndComp
 $EndSCHEMATC
